Commit message: Modifications for making ar_pose working

File: cvg_sim_gazebo/urdf/quadrotor_base.urdf.xacro (robot description, xacro)
@@ -9,5 +9,5 @@
   <!-- Main quadrotor link -->
   <xacro:macro name="quadrotor_base_macro">
-    <link name="base_link">
+    <link name="uav_base_link">
       <inertial>
         <mass value="1.477" />
@@ -28,5 +28,5 @@
       </collision>
     </link>
-    <gazebo reference="base_link">
+    <gazebo reference="uav_base_link">
       <turnGravityOff>false</turnGravityOff>
     </gazebo>

File: cvg_sim_gazebo/urdf/quadrotor_sensors.urdf.xacro (robot description, xacro)
@@ -12,5 +12,5 @@
     <!-- Sonar height sensor -->
     <xacro:include filename="$(find cvg_sim_gazebo)/urdf/sensors/sonar_sensor.urdf.xacro" />
-    <xacro:sonar_sensor name="sonar" parent="base_link" ros_topic="sonar_height" update_rate="10" min_range="0.01" max_range="3.0" field_of_view="${40*M_PI/180}" ray_count="3">
+    <xacro:sonar_sensor name="sonar" parent="uav_base_link" ros_topic="sonar_height" update_rate="10" min_range="0.01" max_range="3.0" field_of_view="${40*M_PI/180}" ray_count="3">
       <origin xyz="-0.15 0.0 0.0" rpy="0 ${90*M_PI/180} 0"/>
     </xacro:sonar_sensor>
@@ -23,10 +23,10 @@
     <!-- Forward facing camera -->
     <xacro:include filename="$(find cvg_sim_gazebo)/urdf/sensors/generic_camera.urdf.xacro" />
-    <xacro:generic_camera name="front" sim_name="ardrone" parent="base_link" update_rate="60" res_x="640" res_y="360" image_format="R8G8B8" hfov="${81*M_PI/180}">
+    <xacro:generic_camera name="front" sim_name="ardrone" parent="uav_base_link" update_rate="60" res_x="640" res_y="360" image_format="R8G8B8" hfov="${81*M_PI/180}">
       <origin xyz="0.21 0.0 0.01" rpy="0 0 0"/>
     </xacro:generic_camera>
     <!-- Downward facing camera -->
     <xacro:include filename="$(find cvg_sim_gazebo)/urdf/sensors/generic_camera.urdf.xacro" />
-    <xacro:generic_camera name="bottom" sim_name="ardrone" parent="base_link" update_rate="60" res_x="640" res_y="360" image_format="R8G8B8" hfov="${81*M_PI/180}">
+    <xacro:generic_camera name="bottom" sim_name="ardrone" parent="uav_base_link" update_rate="60" res_x="640" res_y="360" image_format="R8G8B8" hfov="${81*M_PI/180}">
       <origin xyz="0.15 0.0 0.0" rpy="0 ${M_PI/2} 0"/>
     </xacro:generic_camera>

File: cvg_sim_gazebo/urdf/sensors/generic_camera.urdf.xacro (robot description, xacro)
@@ -82,5 +82,5 @@
           <imageTopicName>/${sim_name}/${name}/image_raw</imageTopicName>
           <cameraInfoTopicName>/${sim_name}/${name}/camera_info</cameraInfoTopicName>
-          <frameName>ardrone_base_${name}cam</frameName>
+          <frameName>/ardrone_base_${name}cam</frameName>
         </plugin>
       </sensor>

File: cvg_sim_gazebo_plugins/urdf/quadrotor_plugins.urdf.xacro (robot description, xacro)
@@ -5,5 +5,5 @@
   <!-- Quadrotor Gazebo Plugins -->
   <xacro:macro name="quadrotor_plugins">
-    <canonicalBody>base_link</canonicalBody>
+    <canonicalBody>uav_base_link</canonicalBody>
     <quadrotor_sensors/>
     <quadrotor_controller/>

File: cvg_sim_gazebo_plugins/urdf/quadrotor_sensors.urdf.xacro (robot description, xacro)
@@ -13,5 +13,5 @@
         <alwaysOn>true</alwaysOn>
         <updateRate>100.0</updateRate>
-        <bodyName>base_link</bodyName>
+        <bodyName>uav_base_link</bodyName>
         <frameId>ardrone_base_link</frameId>
         <topicName>ardrone/imu</topicName>
@@ -37,5 +37,5 @@
         <alwaysOn>true</alwaysOn>
         <updateRate>10.0</updateRate>
-        <bodyName>base_link</bodyName>
+        <bodyName>uav_base_link</bodyName>
         <topicName>pressure_height</topicName>
         <altimeterTopicName>altimeter</altimeterTopicName>
@@ -49,5 +49,5 @@
         <alwaysOn>true</alwaysOn>
         <updateRate>10.0</updateRate>
-        <bodyName>base_link</bodyName>
+        <bodyName>uav_base_link</bodyName>
         <topicName>magnetic</topicName>
         <offset>0.0 0.0 0.0</offset>
@@ -60,5 +60,5 @@
         <alwaysOn>true</alwaysOn>
         <updateRate>4.0</updateRate>
-        <bodyName>base_link</bodyName>
+        <bodyName>uav_base_link</bodyName>
         <topicName>fix</topicName>
         <offset>0.0 0.0 0.0</offset>
@@ -76,5 +76,5 @@
         <alwaysOn>true</alwaysOn>
         <updateRate>100.0</updateRate>
-        <bodyName>base_link</bodyName>
+        <bodyName>uav_base_link</bodyName>
         <topicName>ground_truth/state</topicName>
         <gaussianNoise>0.0</gaussianNoise>

File: cvg_sim_gazebo_plugins/urdf/quadrotor_simple_controller.urdf.xacro (robot description, xacro)
@@ -10,5 +10,5 @@
         <alwaysOn>true</alwaysOn>
         <updateRate>0.0</updateRate>
-        <bodyName>base_link</bodyName>
+        <bodyName>uav_base_link</bodyName>
         <stateTopic>ground_truth/state</stateTopic>
         <imuTopic>ardrone/imu</imuTopic>
@@ -37,5 +37,5 @@
         <alwaysOn>true</alwaysOn>
         <updateRate>0.0</updateRate>
-        <bodyName>base_link</bodyName>
+        <bodyName>uav_base_link</bodyName>
         <stateTopic>ground_truth/state</stateTopic>
         <imuTopic>ardrone/imu</imuTopic>
