Commit message: Added model of husky with marker

File: cvg_sim_gazebo/urdf/husky.gazebo.xacro (robot description, xacro)
@@ -22,67 +22,85 @@
 -->
 <robot name="husky_robot_gazebo" xmlns:xacro="http://ros.org/wiki/xacro">
-  <xacro:include filename="$(find husky_gazebo)/urdf/accessories/kinect_camera.gazebo.xacro"/>
-  <xacro:macro name="husky_robot_gazebo">
-    <gazebo>
-      <plugin name="imu_controller" filename="libhector_gazebo_ros_imu.so">
-        <robotNamespace>/</robotNamespace>
-        <updateRate>50.0</updateRate>
-        <bodyName>base_link</bodyName>
-        <topicName>imu/data</topicName>
-        <accelDrift>0.005 0.005 0.005</accelDrift>
-        <accelGaussianNoise>0.005 0.005 0.005</accelGaussianNoise>
-        <rateDrift>0.005 0.005 0.005 </rateDrift>
-        <rateGaussianNoise>0.005 0.005 0.005 </rateGaussianNoise>
-        <headingDrift>0.005</headingDrift>
-        <headingGaussianNoise>0.005</headingGaussianNoise>
-      </plugin>
-    </gazebo>
-    <gazebo>
-      <plugin name="gps_controller" filename="libhector_gazebo_ros_gps.so">
-        <updateRate>40</updateRate>
-        <robotNamespace>/</robotNamespace>
-        <bodyName>base_link</bodyName>
-        <frameId>base_link</frameId>
-        <topicName>navsat/fix</topicName>
-        <velocityTopicName>navsat/vel</velocityTopicName>
-        <referenceLatitude>49.9</referenceLatitude>
-        <referenceLongitude>8.9</referenceLongitude>
-        <referenceHeading>0</referenceHeading>
-        <referenceAltitude>0</referenceAltitude>
-        <drift>0.0001 0.0001 0.0001</drift>
-      </plugin>
-    </gazebo>
-    <gazebo>
-        <plugin name="gazebo_ros_control" filename="libgazebo_ros_control.so"/>
-          <robotNamespace>/husky</robotNamespace>
-          </plugin>
+    <xacro:include filename="$(find husky_gazebo)/urdf/accessories/kinect_camera.gazebo.xacro"/>
+    <xacro:macro name="husky_robot_gazebo">
+        <gazebo>
+            <plugin name="imu_controller" filename="libhector_gazebo_ros_imu.so">
+                <robotNamespace>/</robotNamespace>
+                <updateRate>50.0</updateRate>
+                <bodyName>base_link</bodyName>
+                <topicName>imu/data</topicName>
+                <gaussianNoise>0</gaussianNoise>
+                <offset>0.0 0.0 0.0</offset>
+                <driftFrequency>0.0 0.0 0.0</driftFrequency>
+                <accelOffset>0 0 0</accelOffset>
+                <accelDrift>0.005 0.005 0.005</accelDrift>
+                <accelDriftFrequency>0.0 0.0 0.0</accelDriftFrequency>
+                <accelGaussianNoise>0.005 0.005 0.005</accelGaussianNoise>
+                <rateOffset>0.0 0.0 0.0</rateOffset>
+                <rateDrift>0.005 0.005 0.005
+                </rateDrift>
+                <rateDriftFrequency>0.0 0.0 0.0</rateDriftFrequency>
+                <rateGaussianNoise>0.005 0.005 0.005
+                </rateGaussianNoise>
+                <headingDrift>0.005</headingDrift>
+                <headingDriftFrequency>0.0</headingDriftFrequency>
+                <headingOffset>0.0</headingOffset>
+                <headingGaussianNoise>0.005</headingGaussianNoise>
+            </plugin>
+        </gazebo>
+        <gazebo>
+            <plugin name="gps_controller" filename="libhector_gazebo_ros_gps.so">
+                <updateRate>40</updateRate>
+                <robotNamespace>/</robotNamespace>
+                <bodyName>base_link</bodyName>
+                <frameId>base_link</frameId>
+                <topicName>navsat/fix</topicName>
+                <offset>0.0 0.0 0.0</offset>
+                <velocityTopicName>navsat/vel</velocityTopicName>
+                <drift>0.0001 0.0001 0.0001</drift>
+                <driftFrequency>0.0 0.0 0.0</driftFrequency>
+                <gaussianNoise>0.0 0.0 0.0</gaussianNoise>
+                <velocityDrift>0 0 0</velocityDrift>
+                <velocityOffset>0 0 0</velocityOffset>
+                <velocityDriftFrequency>0.0 0.0 0.0</velocityDriftFrequency>
+                <velocityGaussianNoise>0.0 0.0 0.0</velocityGaussianNoise>
+                <referenceLatitude>49.9</referenceLatitude>
+                <referenceLongitude>8.9</referenceLongitude>
+                <referenceHeading>0</referenceHeading>
+                <referenceAltitude>0</referenceAltitude>
+            </plugin>
+        </gazebo>
+        <gazebo>
+            <plugin name="gazebo_ros_control" filename="libgazebo_ros_control.so"/>
+            <robotNamespace>/husky</robotNamespace>
+        </plugin>
     </gazebo>
     <xacro:if value="$(arg ur5_enabled)">
-      <!--Remove when https://github.com/ros-industrial/universal_robot/pull/168 is resolved -->
-      <gazebo reference="ur5_arm_shoulder_link">
-        <selfCollide>true</selfCollide>
-      </gazebo>
-      <gazebo reference="ur5_arm_upper_arm_link">
-        <selfCollide>true</selfCollide>
-      </gazebo>
-      <gazebo reference="ur5_arm_forearm_link">
-        <selfCollide>true</selfCollide>
-      </gazebo>
-      <gazebo reference="ur5_arm_wrist_1_link">
-        <selfCollide>true</selfCollide>
-      </gazebo>
-      <gazebo reference="ur5_arm_wrist_3_link">
-       <selfCollide>true</selfCollide>
-      </gazebo>
-      <gazebo reference="ur5_arm_wrist_2_link">
-        <selfCollide>true</selfCollide>
-      </gazebo>
-      <gazebo reference="ur5_arm_ee_link">
-        <selfCollide>true</selfCollide>
-      </gazebo>
+        <!--Remove when https://github.com/ros-industrial/universal_robot/pull/168 is resolved -->
+        <gazebo reference="ur5_arm_shoulder_link">
+            <selfCollide>true</selfCollide>
+        </gazebo>
+        <gazebo reference="ur5_arm_upper_arm_link">
+            <selfCollide>true</selfCollide>
+        </gazebo>
+        <gazebo reference="ur5_arm_forearm_link">
+            <selfCollide>true</selfCollide>
+        </gazebo>
+        <gazebo reference="ur5_arm_wrist_1_link">
+            <selfCollide>true</selfCollide>
+        </gazebo>
+        <gazebo reference="ur5_arm_wrist_3_link">
+            <selfCollide>true</selfCollide>
+        </gazebo>
+        <gazebo reference="ur5_arm_wrist_2_link">
+            <selfCollide>true</selfCollide>
+        </gazebo>
+        <gazebo reference="ur5_arm_ee_link">
+            <selfCollide>true</selfCollide>
+        </gazebo>
     </xacro:if>
     <xacro:if value="$(arg kinect_enabled)">
-      <xacro:kinect_camera_gazebo prefix="camera"/>
+        <xacro:kinect_camera_gazebo prefix="camera"/>
     </xacro:if>
-  </xacro:macro>
+</xacro:macro>
 </robot>

Commit message: MAS ready for experiments

File: cvg_sim_gazebo/urdf/husky.gazebo.xacro (robot description, xacro)
@@ -29,4 +29,5 @@
                 <updateRate>50.0</updateRate>
                 <bodyName>base_link</bodyName>
+                <frameid>husky/base_link</frameid>
                 <topicName>imu/data</topicName>
                 <gaussianNoise>0</gaussianNoise>
@@ -54,5 +55,5 @@
                 <robotNamespace>/</robotNamespace>
                 <bodyName>base_link</bodyName>
-                <frameId>base_link</frameId>
+                <frameId>husky/base_link</frameId>
                 <topicName>navsat/fix</topicName>
                 <offset>0.0 0.0 0.0</offset>

File: cvg_sim_gazebo/urdf/quadrotor_base.urdf.xacro (robot description, xacro)
@@ -9,5 +9,5 @@
   <!-- Main quadrotor link -->
   <xacro:macro name="quadrotor_base_macro">
-    <link name="uav_base_link">
+    <link name="base_link">
       <inertial>
         <mass value="1.477" />
@@ -28,5 +28,5 @@
       </collision>
     </link>
-    <gazebo reference="uav_base_link">
+    <gazebo reference="base_link">
       <turnGravityOff>false</turnGravityOff>
     </gazebo>

File: cvg_sim_gazebo/urdf/quadrotor_sensors.urdf.xacro (robot description, xacro)
@@ -12,5 +12,5 @@
     <!-- Sonar height sensor -->
     <xacro:include filename="$(find cvg_sim_gazebo)/urdf/sensors/sonar_sensor.urdf.xacro" />
-    <xacro:sonar_sensor name="sonar" parent="uav_base_link" ros_topic="sonar_height" update_rate="10" min_range="0.01" max_range="3.0" field_of_view="${40*M_PI/180}" ray_count="3">
+    <xacro:sonar_sensor name="sonar" parent="base_link" ros_topic="sonar_height" update_rate="10" min_range="0.01" max_range="3.0" field_of_view="${40*M_PI/180}" ray_count="3">
       <origin xyz="-0.15 0.0 0.0" rpy="0 ${90*M_PI/180} 0"/>
     </xacro:sonar_sensor>
@@ -23,10 +23,10 @@
     <!-- Forward facing camera -->
     <xacro:include filename="$(find cvg_sim_gazebo)/urdf/sensors/generic_camera.urdf.xacro" />
-    <xacro:generic_camera name="front" sim_name="ardrone" parent="uav_base_link" update_rate="60" res_x="640" res_y="360" image_format="R8G8B8" hfov="${81*M_PI/180}">
+    <xacro:generic_camera name="front" sim_name="ardrone" parent="base_link" update_rate="60" res_x="640" res_y="360" image_format="R8G8B8" hfov="${81*M_PI/180}">
       <origin xyz="0.21 0.0 0.01" rpy="0 0 0"/>
     </xacro:generic_camera>
     <!-- Downward facing camera -->
     <xacro:include filename="$(find cvg_sim_gazebo)/urdf/sensors/generic_camera.urdf.xacro" />
-    <xacro:generic_camera name="bottom" sim_name="ardrone" parent="uav_base_link" update_rate="60" res_x="640" res_y="360" image_format="R8G8B8" hfov="${81*M_PI/180}">
+    <xacro:generic_camera name="bottom" sim_name="ardrone" parent="base_link" update_rate="60" res_x="640" res_y="360" image_format="R8G8B8" hfov="${81*M_PI/180}">
       <origin xyz="0.15 0.0 0.0" rpy="0 ${M_PI/2} 0"/>
     </xacro:generic_camera>

File: cvg_sim_gazebo/urdf/sensors/generic_camera.urdf.xacro (robot description, xacro)
@@ -37,7 +37,7 @@
       <origin xyz="0 0 0" rpy="${-M_PI/2} 0.0 ${-M_PI/2}" />
       <parent link="${name}_link" />
-      <child link="ardrone_base_${name}cam"/>
+      <child link="/ardrone_base_${name}cam"/>
     </joint>
-    <link name="ardrone_base_${name}cam">
+    <link name="/ardrone_base_${name}cam">
       <inertial>
         <mass value="0.01" />

File: cvg_sim_gazebo_plugins/urdf/quadrotor_plugins.urdf.xacro (robot description, xacro)
@@ -5,5 +5,5 @@
   <!-- Quadrotor Gazebo Plugins -->
   <xacro:macro name="quadrotor_plugins">
-    <canonicalBody>uav_base_link</canonicalBody>
+    <canonicalBody>base_link</canonicalBody>
     <quadrotor_sensors/>
     <quadrotor_controller/>

File: cvg_sim_gazebo_plugins/urdf/quadrotor_sensors.urdf.xacro (robot description, xacro)
@@ -13,5 +13,5 @@
         <alwaysOn>true</alwaysOn>
         <updateRate>100.0</updateRate>
-        <bodyName>uav_base_link</bodyName>
+        <bodyName>base_link</bodyName>
         <frameId>ardrone_base_link</frameId>
         <topicName>ardrone/imu</topicName>
@@ -37,5 +37,5 @@
         <alwaysOn>true</alwaysOn>
         <updateRate>10.0</updateRate>
-        <bodyName>uav_base_link</bodyName>
+        <bodyName>base_link</bodyName>
         <topicName>pressure_height</topicName>
         <altimeterTopicName>altimeter</altimeterTopicName>
@@ -49,5 +49,5 @@
         <alwaysOn>true</alwaysOn>
         <updateRate>10.0</updateRate>
-        <bodyName>uav_base_link</bodyName>
+        <bodyName>base_link</bodyName>
         <topicName>magnetic</topicName>
         <offset>0.0 0.0 0.0</offset>
@@ -60,5 +60,5 @@
         <alwaysOn>true</alwaysOn>
         <updateRate>4.0</updateRate>
-        <bodyName>uav_base_link</bodyName>
+        <bodyName>base_link</bodyName>
         <topicName>fix</topicName>
         <offset>0.0 0.0 0.0</offset>
@@ -76,5 +76,5 @@
         <alwaysOn>true</alwaysOn>
         <updateRate>100.0</updateRate>
-        <bodyName>uav_base_link</bodyName>
+        <bodyName>base_link</bodyName>
         <topicName>ground_truth/state</topicName>
         <gaussianNoise>0.0</gaussianNoise>

File: cvg_sim_gazebo_plugins/urdf/quadrotor_simple_controller.urdf.xacro (robot description, xacro)
@@ -10,5 +10,5 @@
         <alwaysOn>true</alwaysOn>
         <updateRate>0.0</updateRate>
-        <bodyName>uav_base_link</bodyName>
+        <bodyName>base_link</bodyName>
         <stateTopic>ground_truth/state</stateTopic>
         <imuTopic>ardrone/imu</imuTopic>
@@ -37,5 +37,5 @@
         <alwaysOn>true</alwaysOn>
         <updateRate>0.0</updateRate>
-        <bodyName>uav_base_link</bodyName>
+        <bodyName>base_link</bodyName>
         <stateTopic>ground_truth/state</stateTopic>
         <imuTopic>ardrone/imu</imuTopic>
